Commit message: Lab 4 and some parts of Lab 3

File: src/my_r2d2/urdf/r2d2_test.urdf.xacro (robot description, xacro)
@@ -35,5 +35,4 @@
       </geometry>
     </collision>
-    <xacro:default_inertial mass="10"/>
   </link>
   <xacro:macro name="wheel" params="prefix suffix reflect">
@@ -52,7 +51,6 @@
         </geometry>
       </collision>
-      <xacro:default_inertial mass="1"/>
-    </link>
-    <joint name="${prefix}_${suffix}_wheel_joint" type="continuous">
+    </link>
+    <joint name="${prefix}_${suffix}_wheel_joint" type="fixed">
       <axis xyz="0 1 0" rpy="0 0 0" />
       <parent link="${prefix}_base"/>
@@ -76,5 +74,4 @@
         <origin xyz="0 0 -${leglen/2}" rpy="0 ${pi/2} 0"/>
       </collision>
-      <xacro:default_inertial mass="10"/>
     </link>
     <joint name="base_to_${prefix}_leg" type="fixed">
@@ -95,5 +92,4 @@
         </geometry>
       </collision>
-      <xacro:default_inertial mass="10"/>
     </link>
     <joint name="${prefix}_base_joint" type="fixed">
@@ -107,5 +103,5 @@
   <xacro:leg prefix="right" reflect="-1" />
   <xacro:leg prefix="left" reflect="1" />
-  <joint name="gripper_extension" type="prismatic">
+  <joint name="gripper_extension" type="fixed">
     <parent link="base_link"/>
     <child link="gripper_pole"/>
@@ -126,8 +122,7 @@
       <origin xyz="${polelen/2} 0 0" rpy="0 ${pi/2} 0 "/>
     </collision>
-    <xacro:default_inertial mass="0.05"/>
   </link>
   <xacro:macro name="gripper" params="prefix reflect">
-    <joint name="${prefix}_gripper_joint" type="revolute">
+    <joint name="${prefix}_gripper_joint" type="fixed">
       <axis xyz="0 0 ${reflect}"/>
       <limit effort="1000.0" lower="0.0" upper="0.548" velocity="0.5"/>
@@ -149,5 +144,4 @@
         <origin rpy="${(reflect-1)/2*pi} 0 0" xyz="0 0 0"/>
       </collision>
-      <xacro:default_inertial mass="0.05"/>
     </link>
     <joint name="${prefix}_tip_joint" type="fixed">
@@ -168,5 +162,4 @@
         <origin rpy="${(reflect-1)/2*pi} 0 0" xyz="0.09137 0.00495 0"/>
       </collision>
-      <xacro:default_inertial mass="0.05"/>
     </link>
   </xacro:macro>
@@ -185,7 +178,6 @@
       </geometry>
     </collision>
-    <xacro:default_inertial mass="2"/>
-  </link>
-  <joint name="head_swivel" type="continuous">
+  </link>
+  <joint name="head_swivel" type="fixed">
     <parent link="base_link"/>
     <child link="head"/>
@@ -206,5 +198,4 @@
       </geometry>
     </collision>
-    <xacro:default_inertial mass="1"/>
   </link>
   <joint name="tobox" type="fixed">
@@ -216,14 +207,23 @@
 <visual>
 <geometry>
-<sphere radius="${width/10}"/>
+<cylinder radius="${width/10}" length="${width/3}"/>
 </geometry>
-<marterial name="black"/>
-<origin xyz="0 0 0"/>
+<origin xyz="${width/15} 0 0" rpy="0 ${pi/2} 0" />
+      <material name="black"/>
 </visual>
 </link>
-<joint name="lensetobox" type="fixed">
+<joint name="lensetoboxX" type="fixed">
+<limit effort="${pi/5}" lower="${-pi/5}" upper="${pi/5}" velocity="0.9"/>
 <parent link="box"/>
 <child link="lense"/>
+<axis xyz="0 0 1"/>
 <origin xyz="0 0 0"/>
 </joint>
+<link name="base_footprint">
+</link>
+<joint name="footprint_base" type="fixed">
+<parent link="base_footprint"/>
+<child link="base_link"/>
+<origin xyz="0 0 ${bodylen/2+0.1+wheeldiam}" rpy="0 0 0"/>
+</joint>
 </robot>
